File: hardware/rotor/Rotor.kicad_pcb (KiCad board)
At the start: 2 copper layers, 200 x 200 mm, 1 part

Commit message: Contacts library
Created a library for the TENG contacts.
Added some footprints for the 10x10cm TENG.
Parts:
- added ?: , , B.Cu at (192.0, 150.0)
- added ?: , , B.Cu at (200.0, 158.0)
- added ?: , , B.Cu at (208.0, 150.0)
- added ?: , , B.Cu at (200.0, 142.0)
- added REF**: PogoPin_D2.0mm, Custom_Parts:PogoPin_D2.0mm, B.Cu at (192.0, 150.0)
- added REF**: PogoPin_D2.0mm, Custom_Parts:PogoPin_D2.0mm, B.Cu at (200.0, 158.0)
- added REF**: PogoPin_D2.0mm, Custom_Parts:PogoPin_D2.0mm, B.Cu at (208.0, 150.0)
- added REF**: PogoPin_D2.0mm, Custom_Parts:PogoPin_D2.0mm, B.Cu at (200.0, 142.0)
- moved G*** 220.0 mm to (-20.0, 207.0)
Other:
- board size 200 x 200 mm -> 370 x 200 mm

Commit message: Generator layouts and footprints
Updated the TENG footprint library.
Updated the rotor and stator PCB layouts.
Generated new 3D models for the rotor and stator.
Parts:
- removed ? (x4): , 
- removed G***: LOGO, TENG:QR
- removed REF** (x4): PogoPin_D2.0mm, Custom_Parts:PogoPin_D2.0mm
- added J1: POGO D2.0mm, TENG:PogoPin_D2.0mm_JOIN, F.Cu at (200.0, 158.0)
- added J10, J11, J12, J5, J6, J7, J8, J9: TENG 10X10 8P, TENG:CONTACT_CIRCLE_10X10_8P, F.Cu at (200.0, 150.0)
- added J2: POGO D2.0mm, TENG:PogoPin_D2.0mm_JOIN, F.Cu at (192.0, 150.0)
- added J3: POGO D2.0mm, TENG:PogoPin_D2.0mm_JOIN, F.Cu at (208.0, 150.0)
- added J4: POGO D2.0mm, TENG:PogoPin_D2.0mm_JOIN, F.Cu at (200.0, 142.0)
Routing:
- net B: track 50.0 -> 0.00 mm, vias 10 -> 0
- net /CON_1: track 0.00 -> 38.1 mm, vias 0 -> 1
- net /CON_3: track 0.00 -> 31.3 mm, vias 0 -> 1
- net /CON_4: track 0.00 -> 29.0 mm, vias 0 -> 2
- net /CON_2: track 0.00 -> 26.9 mm, vias 0 -> 2
- net A: track 15.0 -> 0.00 mm, vias 10 -> 0
- removed copper zone on B.Cu, net A
- removed copper zone on F.Cu, net A
- removed copper zone on B.Cu, net B
- removed copper zone on F.Cu, net B
Other:
- board size 370 x 200 mm -> 100 x 100 mm
- board text removed: "PD 22/04/26"
- board text removed: "REV A"
- board text removed: "TENG ROTOR"
- board text removed: "VERSION 1.0"

Commit message: Pogo pin and production
Changed the pogo pins for ones with greater overall length, this takes into accout the thickness of the dielectric film.
Added the version information to the boards.
Built the production files.
Parts:
- added H1: TOOLING, MountingHole:ToolingHole_1.152mm, F.Cu at (155.6, 149.6)
- added H2: TOOLING, MountingHole:ToolingHole_1.152mm, F.Cu at (200.4, 105.6)
- added H3: TOOLING, MountingHole:ToolingHole_1.152mm, F.Cu at (244.4, 150.4)
- added H4: TOOLING, MountingHole:ToolingHole_1.152mm, F.Cu at (199.6, 194.4)
Other:
- outline, holes or cut-outs redrawn
- board text added: "1"
- board text added: "2"
- board text added: "3"
- board text added: "4"
