File: hardware/stator/Stator.kicad_pcb (KiCad board)
At the start: 2 copper layers, 200 x 200 mm, 1 part

Commit message: Contacts library
Created a library for the TENG contacts.
Added some footprints for the 10x10cm TENG.
Parts:
- added ?: , , F.Cu at (157.0, 107.0)
- added ?: , , F.Cu at (157.0, 193.0)
- added ?: , , F.Cu at (243.0, 193.0)
- added ?: , , B.Cu at (243.0, 107.0)
- added REF**: PogoPin_D2.0mm, Custom_Parts:PogoPin_D2.0mm, F.Cu at (157.0, 193.0)
- added REF**: PogoPin_D2.0mm, Custom_Parts:PogoPin_D2.0mm, F.Cu at (243.0, 193.0)
- added REF**: PogoPin_D2.0mm, Custom_Parts:PogoPin_D2.0mm, F.Cu at (157.0, 107.0)
- added REF**: PogoPin_D2.0mm, Custom_Parts:PogoPin_D2.0mm, F.Cu at (243.0, 107.0)
- moved G*** 220.0 mm to (-20.0, 207.0)
Other:
- board size 200 x 200 mm -> 370 x 200 mm

Commit message: Generator layouts and footprints
Updated the TENG footprint library.
Updated the rotor and stator PCB layouts.
Generated new 3D models for the rotor and stator.
Parts:
- removed ? (x4): , 
- removed G***: LOGO, TENG:QR
- removed REF** (x4): PogoPin_D2.0mm, Custom_Parts:PogoPin_D2.0mm
- added J1: POGO D2.0mm, TENG:PogoPin_D2.0mm_JOIN, F.Cu at (165.0, 107.0)
- added J10, J11, J12, J13, J14, J15, J16, J9: TENG 10X10 8P, TENG:CONTACT_CIRCLE_10X10_8P_HUB, F.Cu at (200.0, 150.0)
- added J2: POGO D2.0mm, TENG:PogoPin_D2.0mm_JOIN, F.Cu at (235.0, 193.0)
- added J3: POGO D2.0mm, TENG:PogoPin_D2.0mm_JOIN, F.Cu at (157.0, 115.0)
- added J4: POGO D2.0mm, TENG:PogoPin_D2.0mm_JOIN, F.Cu at (243.0, 185.0)
- added J5: POGO D2.0mm, TENG:PogoPin_D2.0mm_JOIN, F.Cu at (235.0, 107.0)
- added J6: POGO D2.0mm, TENG:PogoPin_D2.0mm_JOIN, F.Cu at (165.0, 193.0)
- added J7: POGO D2.0mm, TENG:PogoPin_D2.0mm_JOIN, F.Cu at (243.0, 115.0)
- added J8: POGO D2.0mm, TENG:PogoPin_D2.0mm_JOIN, F.Cu at (157.0, 185.0)
Routing:
- net /CON_8: track 0.00 -> 86.6 mm
- net /CON_7: track 0.00 -> 86.6 mm
- net /CON_2: track 0.00 -> 86.6 mm
- net /CON_1: track 0.00 -> 86.6 mm
- net /CON_6: track 0.00 -> 85.7 mm
- net /CON_5: track 0.00 -> 85.7 mm
- net /CON_4: track 0.00 -> 85.7 mm
- net /CON_3: track 0.00 -> 85.7 mm
- net B: track 50.0 -> 0.00 mm, vias 10 -> 0
- net A: track 15.0 -> 0.00 mm, vias 10 -> 0
- removed copper zone on B.Cu, net A
- removed copper zone on F.Cu, net A
- removed copper zone on B.Cu, net B
- removed copper zone on F.Cu, net B
Other:
- board size 370 x 200 mm -> 100 x 100 mm
- board text removed: "PD 22/04/26"
- board text removed: "REV A"
- board text removed: "TENG STATOR"
- board text removed: "VERSION 1.0"

Commit message: Pogo pin and production
Changed the pogo pins for ones with greater overall length, this takes into accout the thickness of the dielectric film.
Added the version information to the boards.
Built the production files.
Parts:
- added H1: TOOLING, MountingHole:ToolingHole_1.152mm, F.Cu at (153.0, 111.0)
- added H2: TOOLING, MountingHole:ToolingHole_1.152mm, F.Cu at (153.0, 189.0)
- added H3: TOOLING, MountingHole:ToolingHole_1.152mm, F.Cu at (247.0, 111.0)
- added H4: TOOLING, MountingHole:ToolingHole_1.152mm, F.Cu at (247.0, 189.0)
Other:
- board text added: "1"
- board text added: "2"
- board text added: "3"
- board text added: "4"
- board text added: "BOTTOM SIDE"
- board text added: "PD 22/04/26"
- board text added: "PD 27/10/2026"
- board text added: "REV A"
- board text added: "TENG STATOR"
- board text added: "TOP SIDE"
- board text added: "V2.0 REV A"
- board text added: "VERSION 1.0"
