File: hardware/stator/Stator.kicad_sch (KiCad schematic)
At the start: 0 parts

Commit message: Generator layouts and footprints
Updated the TENG footprint library.
Updated the rotor and stator PCB layouts.
Generated new 3D models for the rotor and stator.
Parts:
- added J1, J2, J3, J4, J5, J6, J7, J8: POGO D2.0mm, TENG:PogoPin_D2.0mm_JOIN, symbol Connector:Conn_01x01_Pin
- added J10, J11, J12, J13, J14, J15, J16, J9: TENG 10X10 8P, TENG:CONTACT_CIRCLE_10X10_8P_HUB, symbol Connector_Generic:Conn_01x01
Connections:
- new net CON_1: J1.1 (Pin_1), J9.1 (Pin_1)
- new net CON_2: J10.1 (Pin_1), J2.1 (Pin_1)
- new net CON_3: J11.1 (Pin_1), J3.1 (Pin_1)
- new net CON_4: J12.1 (Pin_1), J4.1 (Pin_1)
- new net CON_5: J13.1 (Pin_1), J5.1 (Pin_1)
- new net CON_6: J14.1 (Pin_1), J6.1 (Pin_1)
- new net CON_7: J15.1 (Pin_1), J7.1 (Pin_1)
- new net CON_8: J16.1 (Pin_1), J8.1 (Pin_1)

Commit message: Pogo pin and production
Changed the pogo pins for ones with greater overall length, this takes into accout the thickness of the dielectric film.
Added the version information to the boards.
Built the production files.
Parts:
- added H1, H2, H3, H4: TOOLING, MountingHole:ToolingHole_1.152mm, symbol Mechanical:MountingHole
- J1, J2, J3, J4, J5, J6, J7, J8: JLC Part C20612445 -> C5157421; Manufacturer Part YZ50315020R-03 -> YZ203115028R-03
